File: SpringRobocon2026_mainboard.kicad_sch (KiCad schematic)
At the start: 54 parts, among them J1 Conn_01x05_Socket_Encoder1, J2 Conn_01x05_Socket_Encoder3, J3 FDCAN_1, J4 Conn_01x05_Socket_Encoder2, J5 Conn_01x05_Socket_Encoder4, J6 FDCAN_2, J7 Conn_01x03_Pin, J8 Conn_01x04_Pin, U1 XT60_M, U2 MCP2562-E-P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

Commit message: 回路図更新
Parts:
- added C19: 0.1u, Capacitor_SMD:C_0603_1608Metric_Pad1.08x0.95mm_HandSolder, symbol Device:C
- added J10: Conn_01x05_Socket_Encoder5, MyLib:Pocket_Header_ver, symbol Connector:Conn_01x05_Socket
- added J9: Conn_01x03_Pin, Connector_JST:JST_XH_B3B-XH-A_1x03_P2.50mm_Vertical, symbol Connector:Conn_01x03_Pin
- added R14, R15: 4.7k, Resistor_SMD:R_0603_1608Metric_Pad0.98x0.95mm_HandSolder, symbol Device:R
- added R23, R24: 10k, Resistor_SMD:R_0603_1608Metric_Pad0.98x0.95mm_HandSolder, symbol Device:R
- added SW3: SW_DIP_x02_CANnum, Button_Switch_THT:SW_DIP_SPSTx02_Slide_6.7x6.64mm_W7.62mm_P2.54mm_LowProfile, symbol Switch:SW_DIP_x02
- added U7: XT60_M, Connector_AMASS:AMASS_XT60-M_1x02_P7.20mm_Vertical, symbol Mylib:XT60
Connections:
- net +3V3: now also R23.1, R24.1
- net +5V: now also C19.1, J10.4 (Pin_4), R14.1, R15.1
- net GND: now also C19.2, J10.1 (Pin_1), J9.3 (Pin_3), SW3.3, SW3.4, U7.1
- net PWM_servo: now also J9.1 (Pin_1)
- net En5_B_Tim5_CH2: now reaches U6.CN7_21 (PB7)
- net En5_B_Tim5_CH2: now also J10.5 (Pin_5), R15.2
- net En5_A_Tim5_CH1: now reaches U6.CN10_17 (PB6)
- net En5_A_Tim5_CH1: now also J10.3 (Pin_3), R14.2
- new net +8V: J9.2 (Pin_2), U7.2
- new net board_num1: R23.2, SW3.1
- new net board_num2: R24.2, SW3.2
- no-connect marks 4 -> 5
Other:
- moved on the sheet: C18, D6, D7, D8, J7, J8, R11, R12, R13
