File: SpringRobocon2026_mainboard.kicad_sch (KiCad schematic)
At the start: 63 parts, among them J1 Conn_01x05_Socket_Encoder1, J10 Conn_01x03_Pin, J11 Conn_01x03_Pin, J2 Conn_01x05_Socket_Encoder3, J3 Conn_01x05_Socket_Encoder5, J4 FDCAN_1, J5 Conn_01x05_Socket_Encoder2, J6 Conn_01x05_Socket_Encoder4, J7 FDCAN_2, J8 Conn_01x03_Pin, J9 Conn_01x04_Pin, SW1 SW_DIP_x02_CANnum, U1 XT60_M, U2 ATA6561, U3 BP5293-50, U4 BA033CC0FP, U5 ATA6561, U6 NUCLEO-F446RE

Commit message: PCB編集
Parts:
- removed C17: 0.1u, Capacitor_SMD:C_0603_1608Metric_Pad1.08x0.95mm_HandSolder, symbol Device:C
Changed lines of the file:
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@@
 	(text "SERVO"
 		(exclude_from_sim no)
-		(at 264.414 154.178 0)
+		(at 263.144 153.67 0)
 		(effects
 			(font
@@
 	(wire
 		(pts
-			(xy 278.13 170.18) (xy 278.13 172.72)
-		)
-		(stroke
-			(width 0)
-			(type default)
-		)
-	)
-	(wire
-		(pts
 			(xy 101.6 53.34) (xy 111.76 53.34)
 		)
@@
 	(wire
 		(pts
-			(xy 278.13 180.34) (xy 278.13 182.88)
-		)
-		(stroke
-			(width 0)
-			(type default)
-		)
-	)
-	(wire
-		(pts
 			(xy 149.86 142.24) (xy 149.86 144.78)
 		)
@@
 	(global_label "PWM_servo"
 		(shape input)
-		(at 278.13 170.18 90)
-		(fields_autoplaced yes)
-		(effects
-			(font
-				(size 1.27 1.27)
-			)
-			(justify left)
-		)
-		(property "Intersheetrefs" "${INTERSHEET_REFS}"
-			(at 278.13 157.1143 90)
-			(effects
-				(font
-					(size 1.27 1.27)
-				)
-				(justify left)
-				(hide yes)
-			)
-		)
-	)
-	(global_label "PWM_servo"
-		(shape input)
 		(at 259.08 171.45 0)
 		(fields_autoplaced yes)
@@
 	)
 	(symbol
-		(lib_id "Device:C")
-		(at 278.13 176.53 0)
-		(unit 1)
-		(exclude_from_sim no)
-		(in_bom yes)
-		(on_board yes)
-		(dnp no)
-		(fields_autoplaced yes)
-		(property "Reference" "C17"
-			(at 281.94 175.895 0)
-			(effects
-				(font
-					(size 1.27 1.27)
-				)
-				(justify left)
-			)
-		)
-		(property "Value" "0.1u"
-			(at 281.94 178.435 0)
-			(effects
-				(font
-					(size 1.27 1.27)
-				)
-				(justify left)
-			)
-		)
-		(property "Footprint" "Capacitor_SMD:C_0603_1608Metric_Pad1.08x0.95mm_HandSolder"
-			(at 279.0952 180.34 0)
-			(effects
-				(font
-					(size 1.27 1.27)
-				)
-				(hide yes)
-			)
-		)
-		(property "Datasheet" "~"
-			(at 278.13 176.53 0)
-			(effects
-				(font
-					(size 1.27 1.27)
-				)
-				(hide yes)
-			)
-		)
-		(property "Description" ""
-			(at 278.13 176.53 0)
-			(effects
-				(font
-					(size 1.27 1.27)
-				)
-			)
-		)
-		(pin "1"
-		)
-		(pin "2"
-		)
-		(instances
-			(project "SpringRobocon2026_mainboard"
-				(path "/1ce480f8-d983-42c4-9888-4513037ff8c9"
-					(reference "C17")
-					(unit 1)
-				)
-			)
-		)
-	)
-	(symbol
 		(lib_id "Switch:SW_DIP_x02")
 		(at 273.05 270.51 0)
@@
 					(unit 1)
 				)
-			)
-		)
-	)
-	(symbol
-		(lib_id "power:GND")
-		(at 278.13 182.88 0)
-		(unit 1)
-		(exclude_from_sim no)
-		(in_bom yes)
-		(on_board yes)
-		(dnp no)
-		(property "Reference" "#PWR054"
-			(at 278.13 189.23 0)
-			(effects
-				(font
-					(size 1.27 1.27)
-				)
-				(hide yes)
-			)
-		)
-		(property "Value" "GND"
-			(at 278.13 186.69 0)
-			(effects
-				(font
-					(size 1.27 1.27)
-				)
-			)
-		)
-		(property "Footprint" ""
-			(at 278.13 182.88 0)
-			(effects
-				(font
-					(size 1.27 1.27)
-				)
-				(hide yes)
-			)
-		)
-		(property "Datasheet" ""
-			(at 278.13 182.88 0)
-			(effects
-				(font
-					(size 1.27 1.27)
-				)
-				(hide yes)
-			)
-		)
-		(property "Description" ""
-			(at 278.13 182.88 0)
-			(effects
-				(font
-					(size 1.27 1.27)
-				)
-			)
-		)
-		(pin "1"
-		)
-		(instances
-			(project "SpringRobocon2026_mainboard"
-				(path "/1ce480f8-d983-42c4-9888-4513037ff8c9"
-					(reference "#PWR054")
-					(unit 1)
-				)

Commit message: 配線始まり
Parts:
- added C17: 0.1u, Capacitor_SMD:C_0603_1608Metric_Pad1.08x0.95mm_HandSolder, symbol Device:C
- added D6: GS1010FL, Diode_SMD:D_SOD-123F, symbol Device:D
- added J8: SOLENOID1, Connector_JST:JST_XH_B2B-XH-A_1x02_P2.50mm_Vertical, symbol Connector:Conn_01x02_Socket
- added Q1: MTA100N10KRI3, Package_TO_SOT_THT:TO-251-3_Vertical, symbol MyLib:MTA100N10KRI3
- added R13: 1k, Resistor_SMD:R_0603_1608Metric_Pad0.98x0.95mm_HandSolder, symbol Device:R
- added R15: 10k, Resistor_SMD:R_0603_1608Metric_Pad0.98x0.95mm_HandSolder, symbol Device:R
- renumbered D6 to D7, D7 to D8, D8 to D9, J9 to J10, J10 to J11, J11 to J12, J8 to J9, R13 to R14, R14 to R16, R15 to R17, R16 to R18, R17 to R19
Connections:
- net +12V: now also C17.1, D6.1 (K), J8.1 (Pin_1)
- net GND: now also C17.2, Q1.3 (S), R15.2
- net PWM_servo: now also U6.CN7_28 (PA0)
- net SOLENOID: now reaches U6.CN7_35 (PC2)
- net SOLENOID: now also R13.1
- new net: Q1.1 (G), R13.2, R15.1
- new net: D6.2 (A), J8.2 (Pin_2), Q1.2 (D)
- no-connect marks 41 -> 39
Other:
- note added: "SOLENOID"
- moved on the sheet: J9
