File: SpringRobocon2026_mainboard.kicad_sch (KiCad schematic)
At the start: 68 parts, among them J1 Conn_01x05_Socket_Encoder1, J10 Conn_01x04_Pin, J11 Conn_01x03_Pin, J12 Conn_01x03_Pin, J2 Conn_01x05_Socket_Encoder3, J3 Conn_01x05_Socket_Encoder5, J4 FDCAN_1, J5 Conn_01x05_Socket_Encoder2, J6 Conn_01x05_Socket_Encoder4, J7 FDCAN_2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

Commit message: 3回目修正
Connections:
- net +12V: now also D1.2 (A), F1.2; no longer F1.1, U1.2
- net +3V3 renamed +3.3V
- new net: F1.1, U1.2
Other:
- moved on the sheet: C14, C15, C16, D4, F1, U1, U4
