File: SpringRobocon2026_mainboard.kicad_pcb (KiCad board)
At the start: 2 copper layers, 100 x 100 mm, 63 parts, among them J1 Conn_01x05_Socket_Encoder1, J10 Conn_01x03_Pin, J11 Conn_01x03_Pin, J2 Conn_01x05_Socket_Encoder3, J3 Conn_01x05_Socket_Encoder5, J4 FDCAN_1, J5 Conn_01x05_Socket_Encoder2, J6 Conn_01x05_Socket_Encoder4, J7 FDCAN_2, J8 Conn_01x03_Pin, J9 Conn_01x04_Pin, SW1 SW_DIP_x02_CANnum, U1 XT60_M, U2 ATA6561, U3 BP5293-50, U4 BA033CC0FP, U5 ATA6561, U6 NUCLEO-F446RE

Commit message: PCB編集
Parts:
- removed C17: 0.1u, Capacitor_SMD:C_0603_1608Metric_Pad1.08x0.95mm_HandSolder
- added REF**: MountingHole_3.2mm_M3, MountingHole:MountingHole_3.2mm_M3, F.Cu at (90.5, 137.0)
- added REF**: MountingHole_3.2mm_M3, MountingHole:MountingHole_3.2mm_M3, F.Cu at (184.5, 137.0)
- added REF**: MountingHole_3.2mm_M3, MountingHole:MountingHole_3.2mm_M3, F.Cu at (90.5, 43.0)
- added REF**: MountingHole_3.2mm_M3, MountingHole:MountingHole_3.2mm_M3, F.Cu at (184.5, 43.0)
- D2: moved to B.Cu
- moved U1 173.9 mm to (152.5, 131.8), turned to 90 degrees
- moved C12 170.1 mm to (224.7, 64.4)
- moved C11 170.1 mm to (220.4, 84.5)
- moved C2 170.1 mm to (220.4, 66.9)
- moved C3 170.1 mm to (220.4, 69.4)
- moved C4 170.1 mm to (220.4, 71.9)
- moved J1 170.1 mm to (226.6, 28.6)
- moved J2 170.1 mm to (226.6, 36.6)
- moved J3 170.1 mm to (226.6, 44.5)
- moved J5 170.1 mm to (226.6, 52.5)
- moved J6 170.1 mm to (226.6, 60.4)
- moved R1 169.9 mm to (224.7, 79.5)
- moved R2 169.9 mm to (224.7, 82.0)
- moved R10 169.9 mm to (229.1, 79.5)
- moved R11 169.9 mm to (229.1, 82.0)
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
Commit message: 配線始まり
Parts:
- added C17: 0.1u, Capacitor_SMD:C_0603_1608Metric_Pad1.08x0.95mm_HandSolder, B.Cu at (97.8, 110.9)
- added D6: GS1010FL, Diode_SMD:D_SOD-123F, B.Cu at (91.0, 109.4)
- added J8: SOLENOID1, Connector_JST:JST_XH_B2B-XH-A_1x02_P2.50mm_Vertical, F.Cu at (94.8, 110.8)
- added Q1: MTA100N10KRI3, Package_TO_SOT_THT:TO-251-3_Vertical, F.Cu at (93.1, 103.6)
- added R13: 1k, Resistor_SMD:R_0603_1608Metric_Pad0.98x0.95mm_HandSolder, B.Cu at (93.3, 100.5)
- added R15: 10k, Resistor_SMD:R_0603_1608Metric_Pad0.98x0.95mm_HandSolder, B.Cu at (97.0, 101.2)
- C11, C12, C14, C15, C18, C19, C2, C3, C4, C7, C8, D1, D3, D4, D5, R1, R10, R11, R2, R3, R4, R5, R6, R8, R9, U4: moved to B.Cu
- R14: renamed from R13; moved to B.Cu
- R16: renamed from R14; moved to B.Cu
- R17: renamed from R15; moved to B.Cu
- R18: renamed from R16; moved to B.Cu
- R19: renamed from R17; moved to B.Cu
- moved C1 136.3 mm to (178.2, 65.4)
- moved C10 136.1 mm to (178.7, 80.4)
- moved U5 134.2 mm to (174.8, 77.0)
- moved U2 133.1 mm to (174.6, 62.0)
- moved J7 128.0 mm to (184.4, 76.4), turned to -90 degrees
- moved J4 127.8 mm to (184.4, 59.7), turned to -90 degrees
- moved C13 127.4 mm to (170.2, 77.0), turned to 90 degrees
- moved R12 127.0 mm to (179.4, 77.2), turned to -90 degrees
- moved R7 126.2 mm to (179.2, 61.8), turned to -90 degrees
- moved C5 125.3 mm to (170.0, 62.0), turned to 90 degrees
- moved J5 120.1 mm to (118.4, 104.6), turned to 180 degrees
- moved R10 117.7 mm to (114.2, 104.7), turned to 180 degrees
- moved R8 115.5 mm to (117.7, 104.7)
- moved C11 108.0 mm to (115.0, 108.3), turned to 180 degrees
- moved J2 103.2 mm to (151.3, 107.0), turned to -90 degrees
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- renumbered D6 to D7, D7 to D8, D8 to D9, J9 to J10, J10 to J11, J11 to J12, J8 to J9
Connections:
- U6 pad CN7_28: unconnected-(U6A-PA0-PadCN7_28) -> PWM_servo
- U6 pad CN7_35: unconnected-(U6A-PC2-PadCN7_35) -> SOLENOID
Routing:
- net +5V: track 0.00 -> 97.4 mm
- net +3V3: track 0.00 -> 96.0 mm, vias 0 -> 6
- net +12V: track 0.00 -> 31.2 mm
- net Net-(D1-K): track 0.00 -> 18.3 mm
- net SOLENOID: track 0.00 -> 11.6 mm
- net Net-(D6-A): track 0.00 -> 8.86 mm
- net Net-(D1-A): track 0.00 -> 5.37 mm
- net Net-(Q1-G): track 0.00 -> 5.16 mm
- net Net-(D7-A): track 0.00 -> 4.52 mm
