File: SpringRobocon2026_mainboard.kicad_pcb (KiCad board)
At the start: 2 copper layers, 100 x 100 mm, 72 parts, among them J1 Conn_01x05_Socket_Encoder1, J10 Conn_01x04_Pin, J11 Conn_01x03_Pin, J12 Conn_01x03_Pin, J2 Conn_01x05_Socket_Encoder3, J3 Conn_01x05_Socket_Encoder5, J4 FDCAN_1, J5 Conn_01x05_Socket_Encoder2, J6 Conn_01x05_Socket_Encoder4, J7 FDCAN_2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

Commit message: 配線更新
Parts:
- moved R18 1.90 mm to (133.2, 127.9)
- moved D8 1.37 mm to (127.9, 130.3)
- moved R10 1.36 mm to (120.5, 120.1)
- moved R8 1.36 mm to (123.9, 120.1)
- moved R5 1.32 mm to (167.0, 103.5)
- moved R11 1.28 mm to (137.4, 120.2)
- moved R2 1.28 mm to (166.9, 106.9)
- moved R9 1.25 mm to (141.1, 120.2)
- moved R6 1.12 mm to (175.1, 102.9)
- moved R3 1.12 mm to (175.1, 106.5)
- moved R1 1.05 mm to (184.3, 106.4)
- moved R4 1.01 mm to (184.3, 102.8)
- moved C2 0.96 mm to (178.8, 104.8)
- moved C11 0.77 mm to (121.3, 125.8)
- moved C3 0.60 mm to (161.1, 104.3)
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Routing:
- net En5_A_Tim8_CH1: track 0.00 -> 62.5 mm, vias 0 -> 2
- net SDA: track 0.00 -> 61.5 mm
- net SCL: track 0.00 -> 61.5 mm
- net En3_A_Tim3_CH1: track 0.00 -> 48.9 mm
- net En1_A_Tim1_CH1: track 0.00 -> 43.1 mm, vias 0 -> 2
- net En5_B_Tim8_CH2: track 0.00 -> 41.5 mm, vias 0 -> 1
- net En1_B_Tim1_CH2: track 0.00 -> 39.4 mm
- net En3_B_Tim3_CH2: track 0.00 -> 37.4 mm
- net PWM_2: track 0.00 -> 23.2 mm, vias 0 -> 1
- net FDCAN_2TX: track 0.00 -> 15.3 mm
- net En2_B_Tim2_CH2: track 47.5 -> 40.2 mm
- net FDCAN_1TX: track 0.00 -> 7.27 mm
- net FDCAN_1RX: track 0.00 -> 6.74 mm
- net En2_A_Tim2_CH1: track 1.87 -> 0.24 mm
- net En4_B_Tim4_CH2: track 0.00 -> 0.79 mm
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Other:
- board text added: "${REFERENCE}"

Commit message: 一旦完成
Parts:
- added ref**: val**, MyLib:ROGIKEN, F.Cu at (177.2, 131.0)
- moved J12 14.1 mm to (174.1, 75.0)
- moved U5 11.5 mm to (175.0, 88.5)
- moved C13 11.4 mm to (170.4, 88.3)
- moved C10 11.4 mm to (178.9, 91.8)
- moved J7 11.4 mm to (184.6, 87.8)
- moved R12 11.4 mm to (179.6, 88.5)
- moved C1 0.60 mm to (178.2, 66.0)
- moved U2 0.11 mm to (174.5, 62.1)
Routing:
- net board_num1: track 0.00 -> 98.3 mm, vias 0 -> 2
- net board_num2: track 0.00 -> 95.2 mm, vias 0 -> 3
- net En2_A_Tim2_CH1: track 0.24 -> 65.9 mm, vias 0 -> 1
- net En4_B_Tim4_CH2: track 0.79 -> 65.1 mm, vias 0 -> 1
- net En4_A_Tim4_CH1: track 0.00 -> 63.8 mm, vias 0 -> 2
- net FDCAN_2RX: track 0.00 -> 31.1 mm, vias 0 -> 1
- net PWM_2: track 23.2 -> 8.65 mm, vias 1 -> 0
- net DIR_2: track 0.00 -> 8.56 mm
- net En2_B_Tim2_CH2: track 40.2 -> 48.4 mm
- net FDCAN_2TX: track 15.3 -> 7.43 mm, vias 0 -> 1
- net Net-(J4-Pin_1): track 0.00 -> 7.79 mm
- net Net-(J7-Pin_2): track 0.00 -> 7.42 mm
- net Net-(J4-Pin_2): track 0.00 -> 7.34 mm
- net Net-(J7-Pin_1): track 0.00 -> 6.98 mm
- net GND: track 0.00 -> 3.95 mm, vias 0 -> 919
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- added copper zone on B.Cu, net GND
- added copper zone on F.Cu, net GND
Other:
- board text added: "12V"
- board text added: "12V Only!"
- board text added: "12V_IN"
- board text added: "3.3V"
- board text added: "5V"
- board text added: "B 5V A X GND"
- board text added: "CAN1"
- board text added: "CAN2"
- board text added: "DC1"
- board text added: "DC2"
- board text added: "DIR PWM GND"
- board text added: "En_1_Tim1"
- board text added: "En_2_Tim2"
- board text added: "En_3_Tim3"
- board text added: "En_4_Tim4"
- board text added: "En_5_Tim8"
- board text added: "GND 5V SCL SDA"
- board text added: "GND X A 5V B"
- board text added: "PWM GND GND"
- board text added: "R9"
- board text added: "SENSOR"
- board text added: "SERVO"
- board text added: "SOLENOID"
- board text added: "SpringRobocon2026_mainboard"
- board text added: "board_num"
- board text removed: "${REFERENCE}"
