File: SpringRobocon2026_mainboard.kicad_pcb (KiCad board)
At the start: 2 copper layers, 100 x 100 mm, 74 parts, among them J1 Conn_01x05_Socket_Encoder1, J10 Conn_01x04_Pin, J11 Conn_01x03_Pin, J12 Conn_01x03_Pin, J2 Conn_01x05_Socket_Encoder3, J3 Conn_01x05_Socket_Encoder5, J4 FDCAN_1, J5 Conn_01x05_Socket_Encoder2, J6 Conn_01x05_Socket_Encoder4, J7 FDCAN_2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

Commit message: 6回目修正
Parts:
- moved D7 14.3 mm to (92.8, 126.3)
- moved R17 10.3 mm to (93.5, 120.0)
- moved D1 9.19 mm to (108.1, 106.5)
- moved U1 4.03 mm to (106.1, 132.2)
- moved F1 3.78 mm to (97.3, 124.0)
- moved C6 3.25 mm to (112.2, 106.8), turned to -90 degrees
Routing:
- net +12V: track 24.5 -> 47.1 mm
- net Net-(D1-K): track 17.5 -> 11.6 mm
- net +5V: track 313.2 -> 317.2 mm
- net GND: vias 1044 -> 1029
